Commit message: alot again.... adjusting environment and implementing webot functions. Next steps: testing/ debugging environment and testing that the functions of the Webot simulation are callable

File: controllers/RL_Controller/ur5e.urdf (robot description, URDF)
Before this commit: robot ur5e_robot, 11 links, 10 joints
Joints:
- joint elbow_joint: limit lower=-3.141592653589793 upper=3.141592653589793 effort=150.0 velocity=3.141592653589793 -> lower=-6.283185307179586 upper=6.283185307179586 effort=150.0 velocity=3.141592653589793
