Commit message: simplefyed and added controller1

File: controllers/controller_test/ur5e.urdf (robot description, URDF)
Before this commit: robot ur5e_robot, 11 links, 10 joints
Links:
- removed link base_link_inertia
- removed link flange
- added link ee_link; collision box size=0.01 0.01 0.01
- added link world
- link base_link: mass None -> 4.0; geometry collision mesh filename=../meshes/ur5e/collision/base.stl scale=1.0 1.0 1.0; visual mesh filename=../meshes/ur5e/visual/base.dae
- link forearm_link: geometry collision mesh filename=../meshes/ur5e/collision/forearm.stl scale=1.0 1.0 1.0; visual mesh filename=../meshes/ur5e/visual/forearm.dae
- link shoulder_link: geometry collision mesh filename=../meshes/ur5e/collision/shoulder.stl scale=1.0 1.0 1.0; visual mesh filename=../meshes/ur5e/visual/shoulder.dae
- link upper_arm_link: geometry collision mesh filename=../meshes/ur5e/collision/upperarm.stl scale=1.0 1.0 1.0; visual mesh filename=../meshes/ur5e/visual/upperarm.dae
- link wrist_1_link: geometry collision mesh filename=../meshes/ur5e/collision/wrist1.stl scale=1.0 1.0 1.0; visual mesh filename=../meshes/ur5e/visual/wrist1.dae
- link wrist_2_link: geometry collision mesh filename=../meshes/ur5e/collision/wrist2.stl scale=1.0 1.0 1.0; visual mesh filename=../meshes/ur5e/visual/wrist2.dae
- link wrist_3_link: geometry collision mesh filename=../meshes/ur5e/collision/wrist3.stl scale=1.0 1.0 1.0; visual mesh filename=../meshes/ur5e/visual/wrist3.dae
Joints:
- removed joint base_link-base_link_inertia
- removed joint flange-tool0
- removed joint wrist_3-flange
- added joint ee_fixed_joint: type fixed, parent wrist_3_link, child ee_link, origin xyz=0.0 0.1 0.0 rpy=0.0 0.0 1.57079632679
- added joint world_joint: type fixed, parent world, child base_link, origin xyz=0.0 0.0 0.0 rpy=0.0 0.0 0.0
- added joint wrist_3_link-tool0_fixed_joint: type fixed, parent wrist_3_link, child tool0, origin xyz=0 0.1 0 rpy=-1.57079632679 0 0
- joint base_link-base_fixed_joint: origin xyz=0 0 0 rpy=0 0 3.141592653589793 -> xyz=0 0 0 rpy=0 0 -3.14159265359
- joint elbow_joint: axis 0 0 1 -> 0 1 0; limit lower=-6.283185307179586 upper=6.283185307179586 effort=150.0 velocity=3.141592653589793 -> lower=-3.14159265359 upper=3.14159265359 effort=150.0 velocity=3.14; origin xyz=-0.425 0 0 rpy=0 0 0 -> xyz=0.0 -0.131 0.425 rpy=0.0 0.0 0.0
- joint shoulder_lift_joint: axis 0 0 1 -> 0 1 0; limit lower=-6.283185307179586 upper=6.283185307179586 effort=150.0 velocity=3.141592653589793 -> lower=-6.28318530718 upper=6.28318530718 effort=150.0 velocity=3.14; origin xyz=0 0 0 rpy=1.570796327 0 0 -> xyz=0.0 0.138 0.0 rpy=0.0 1.57079632679 0.0
- joint shoulder_pan_joint: limit lower=-6.283185307179586 upper=6.283185307179586 effort=150.0 velocity=3.141592653589793 -> lower=-6.28318530718 upper=6.28318530718 effort=150.0 velocity=3.14; origin xyz=0 0 0.1625 rpy=0 0 0 -> xyz=0.0 0.0 0.163 rpy=0.0 0.0 0.0; parent base_link_inertia -> base_link
- joint wrist_1_joint: axis 0 0 1 -> 0 1 0; limit lower=-6.283185307179586 upper=6.283185307179586 effort=28.0 velocity=3.141592653589793 -> lower=-6.28318530718 upper=6.28318530718 effort=28.0 velocity=6.28; origin xyz=-0.3922 0 0.1333 rpy=0 0 0 -> xyz=0.0 0.0 0.392 rpy=0.0 1.57079632679 0.0
- joint wrist_2_joint: limit lower=-6.283185307179586 upper=6.283185307179586 effort=28.0 velocity=3.141592653589793 -> lower=-6.28318530718 upper=6.28318530718 effort=28.0 velocity=6.28; origin xyz=0 -0.0997 -2.044881182297852e-11 rpy=1.570796327 0 0 -> xyz=0.0 0.127 0.0 rpy=0.0 0.0 0.0
- joint wrist_3_joint: axis 0 0 1 -> 0 1 0; limit lower=-6.283185307179586 upper=6.283185307179586 effort=28.0 velocity=3.141592653589793 -> lower=-6.28318530718 upper=6.28318530718 effort=28.0 velocity=6.28; origin xyz=0 0.0996 -2.042830148012698e-11 rpy=1.570796326589793 3.141592653589793 3.141592653589793 -> xyz=0.0 0.0 0.1 rpy=0.0 0.0 0.0
